File: SMA_Test_Bed/Quad_Current_Driver.kicad_sch (KiCad schematic)
At the start: 38 parts, among them J6 Conn_01x02_Socket, J7 Conn_01x02_Socket, J8 Conn_01x02_Socket, J9 Conn_01x02_Socket, Q5 NMOS, Q6 NMOS, Q7 NMOS, Q8 NMOS, U3 TLV9044

Commit message: Added passive values
Parts:
- C13, C14, C17, C18: value C -> 270nF
- R21, R22, R31, R32: value R_US -> 3Meg
- R23, R24, R33, R34: value R_US -> 470k
- R27, R28, R37, R38: value R_US -> 100
- R29, R30, R39, R40: value R_US -> 5
Changed lines of the file:
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@@
 			)
 		)
-		(property "Value" "C"
+		(property "Value" "270nF"
 			(at 77.47 64.7699 0)
 			(effects
@@
 			)
 		)
-		(property "Value" "R_US"
+		(property "Value" "470k"
 			(at 190.5 137.1599 0)
 			(effects
@@
 			)
 		)
-		(property "Value" "R_US"
+		(property "Value" "5"
 			(at 247.65 68.5799 0)
 			(effects
@@
 			)
 		)
-		(property "Value" "C"
+		(property "Value" "270nF"
 			(at 203.2 137.1599 0)
 			(effects
@@
 			)
 		)
-		(property "Value" "R_US"
+		(property "Value" "100"
 			(at 104.14 119.38 90)
 			(effects
@@
 			)
 		)
-		(property "Value" "R_US"
+		(property "Value" "3Meg"
 			(at 54.356 131.318 90)
 			(effects
@@
 			)
 		)
-		(property "Value" "R_US"
+		(property "Value" "470k"
 			(at 64.77 64.7699 0)
 			(effects
@@
 			)
 		)
-		(property "Value" "R_US"
+		(property "Value" "5"
 			(at 121.92 135.8899 0)
 			(effects
@@
 			)
 		)
-		(property "Value" "R_US"
+		(property "Value" "470k"
 			(at 190.5 67.3099 0)
 			(effects
@@
 			)
 		)
-		(property "Value" "R_US"
+		(property "Value" "100"
 			(at 104.14 49.53 90)
 			(effects
@@
 			)
 		)
-		(property "Value" "R_US"
+		(property "Value" "470k"
 			(at 64.77 134.6199 0)
 			(effects
@@
 			)
 		)
-		(property "Value" "R_US"
+		(property "Value" "3Meg"
 			(at 180.086 133.858 90)
 			(effects
@@
 			)
 		)
-		(property "Value" "R_US"
+		(property "Value" "100"
 			(at 229.87 121.92 90)
 			(effects
@@
 			)
 		)
-		(property "Value" "C"
+		(property "Value" "270nF"
 			(at 203.2 67.3099 0)
 			(effects
@@
 			)
 		)
-		(property "Value" "R_US"
+		(property "Value" "3Meg"
 			(at 54.356 61.468 90)
 			(effects
@@
 			)
 		)
-		(property "Value" "C"
+		(property "Value" "270nF"
 			(at 77.47 134.6199 0)
 			(effects
@@
 			)
 		)
-		(property "Value" "R_US"
+		(property "Value" "5"
 			(at 121.92 66.0399 0)
 			(effects
@@
 			)
 		)
-		(property "Value" "R_US"
+		(property "Value" "5"
 			(at 247.65 138.4299 0)
 			(effects
@@
 			)
 		)
-		(property "Value" "R_US"
+		(property "Value" "3Meg"
 			(at 180.086 64.008 90)
 			(effects
@@
 			)
 		)
-		(property "Value" "R_US"
+		(property "Value" "100"
 			(at 229.87 52.07 90)
 			(effects

Commit message: Time of fabrication
Parts:
- added R84, R88, R92, R96: 100k, Resistor_SMD:R_0603_1608Metric, symbol Device:R_US
- C12, C15, C16, C19, C20: value C -> 100nF; Digikey PN (none) -> 311-1088-1-ND
- C13, C14, C17, C18: Digikey PN (none) -> 490-16405-1-ND
- Q5, Q6, Q7, Q8: footprint Package_TO_SOT_SMD:SOT-23-3 -> Package_TO_SOT_SMD:SOT-223; symbol Simulation_SPICE:NMOS -> Device:Q_NMOS_GDSD; Digikey PN (none) -> DMN3032LE-13DICT-ND
- R21, R22, R31, R32: Digikey PN (none) -> RMCF0603FT3M00CT-ND
- R23, R24, R33, R34: Digikey PN (none) -> YAG4560CT-ND
- R25, R26, R35, R36: value R_US -> 10k; Digikey PN (none) -> 311-10.0KHRCT-ND
- R27, R28, R37, R38: value 100 -> 1k; Digikey PN (none) -> 311-1.00KHRCT-ND
- R29, R30, R39, R40: value 5 -> 5.1; Digikey PN (none) -> A103115CT-ND
- U3: Digikey PN (none) -> 296-TLV9044IDRCT-ND
Connections:
- net +3.3V: no longer J6.1 (Pin_1), J7.1 (Pin_1), J8.1 (Pin_1), J9.1 (Pin_1)
- net GND: now also R84.1, R88.1, R92.1, R96.1
- net at Q8.1 (G): now also R38.2, R96.2; no longer J9.2 (Pin_2)
- net at Q8.2 (D): now also J9.2 (Pin_2), Q8.4 (D); no longer R38.2
- net at J6.2 (Pin_2): now also Q5.2 (D), Q5.4 (D); no longer Q5.1 (D)
- net at R28.2: now also Q6.1 (G), R88.2; no longer Q6.2 (G)
- net at J7.2 (Pin_2): now also Q6.2 (D), Q6.4 (D); no longer Q6.1 (D)
- net at R27.2: now also Q5.1 (G), R84.2; no longer Q5.2 (G)
- net at Q7.1 (G): now also R37.2, R92.2; no longer J8.2 (Pin_2)
- net at Q7.2 (D): now also J8.2 (Pin_2), Q7.4 (D); no longer R37.2
- new net Vdrive: J6.1 (Pin_1), J7.1 (Pin_1), J8.1 (Pin_1), J9.1 (Pin_1)
Other:
- moved on the sheet: J6, J7, J8, J9, R29, R30, R39, R40
