File: SMA_Test_Bed/SMA_Test_Bed.kicad_pcb (KiCad board)
At the start: 2 copper layers, 108.6 x 58.3 mm, 157 parts, among them J1 Conn_02x14_Counter_Clockwise, J10 Conn_01x02_Socket, J11 Conn_01x02_Socket, J12 Conn_01x02_Socket, J13 Conn_01x02_Socket, J14 Conn_01x02_Socket, J15 Conn_01x02_Socket, J16 Conn_01x02_Socket, J17 Conn_01x02_Socket, J18 Conn_01x02_Socket, J2 Conn_01x02_Socket, J3 Conn_01x02_Socket, J4 Conn_01x02_Socket, J5 Conn_01x02_Socket, J6 Conn_01x02_Socket, J7 Conn_01x02_Socket, J8 Conn_01x02_Socket, J9 Conn_01x02_Socket, Q1 NMOS, Q10 NMOS, Q11 NMOS, Q12 NMOS, Q13 NMOS, Q14 NMOS, Q15 NMOS, Q16 NMOS, Q2 NMOS, Q3 NMOS, Q4 NMOS, Q5 NMOS, Q6 NMOS, Q7 NMOS, Q8 NMOS, Q9 NMOS, U1 PCA9685PW, U2 TLV9044, U3 TLV9044, U4 TLV9044, U5 TLV9044

Commit message: Layout draft complete
Parts:
- added H1: MountingHole, MountingHole:MountingHole_2.7mm_Pad_Via, F.Cu at (180.6, 79.5)
- added H2: MountingHole, MountingHole:MountingHole_2.7mm_Pad_Via, F.Cu at (127.1, 79.5)
- added H3: MountingHole, MountingHole:MountingHole_2.7mm_Pad_Via, F.Cu at (108.6, 125.9)
- added H4: MountingHole, MountingHole:MountingHole_2.7mm_Pad_Via, F.Cu at (194.0, 122.4)
- added R81: R_US, Resistor_SMD:R_0603_1608Metric, F.Cu at (137.5, 113.6)
- added R82: R_US, Resistor_SMD:R_0603_1608Metric, F.Cu at (139.6, 113.6)
- moved J18 6.43 mm to (191.8, 114.2)
Routing:
- net +3.3V: track 72.7 -> 61.0 mm, vias 12 -> 8
- net /SCL: track 31.7 -> 36.7 mm, vias 1 -> 2
- net /SDA: track 33.8 -> 37.1 mm, vias 2 -> 3
- net /bus2.PWM_SP3: track 76.5 -> 77.7 mm, vias 2 -> 4
- net /bus2.PWM_SP2: track 64.4 -> 65.2 mm, vias 4 -> 6
- net Net-(C10-Pad2): track 22.7 -> 21.9 mm, vias 1 -> 0
- net /bus1.PWM_SP1: track 89.3 -> 89.9 mm
- net Net-(C7-Pad2): vias 1 -> 0
- net Net-(C37-Pad2): vias 1 -> 0
- net Net-(C34-Pad2): vias 1 -> 0
- net Net-(C28-Pad2): vias 1 -> 0
- net Net-(C25-Pad2): vias 1 -> 0
- net Net-(C19-Pad2): vias 1 -> 0
- net Net-(C16-Pad2): vias 1 -> 0
Other:
- board size 108.6 x 58.3 mm -> 108.6 x 58.4 mm

Commit message: Time of fabrication
Parts:
- added R83: 100k, Resistor_SMD:R_0603_1608Metric, F.Cu at (135.0, 79.6)
- added R84: 100k, Resistor_SMD:R_0603_1608Metric, F.Cu at (197.2, 79.7)
- added R85: 100k, Resistor_SMD:R_0603_1608Metric, F.Cu at (166.4, 79.6)
- added R86: 100k, Resistor_SMD:R_0603_1608Metric, F.Cu at (103.6, 79.6)
- added R87: 100k, Resistor_SMD:R_0603_1608Metric, F.Cu at (155.0, 91.3)
- added R88: 100k, Resistor_SMD:R_0603_1608Metric, F.Cu at (217.2, 91.3)
- added R89: 100k, Resistor_SMD:R_0603_1608Metric, F.Cu at (186.4, 91.3)
- added R90: 100k, Resistor_SMD:R_0603_1608Metric, F.Cu at (123.6, 91.3)
- added R91: 100k, Resistor_SMD:R_0603_1608Metric, F.Cu at (135.1, 87.1)
- added R92: 100k, Resistor_SMD:R_0603_1608Metric, F.Cu at (197.2, 87.2)
- added R93: 100k, Resistor_SMD:R_0603_1608Metric, F.Cu at (166.4, 87.1)
- added R94: 100k, Resistor_SMD:R_0603_1608Metric, F.Cu at (103.7, 87.1)
- added R95: 100k, Resistor_SMD:R_0603_1608Metric, F.Cu at (155.0, 83.8)
- added R96: 100k, Resistor_SMD:R_0603_1608Metric, F.Cu at (217.2, 83.8)
- added R97: 100k, Resistor_SMD:R_0603_1608Metric, F.Cu at (186.4, 83.8)
- added R98: 100k, Resistor_SMD:R_0603_1608Metric, F.Cu at (123.6, 83.8)
- C10, C11, C12, C15, C16, C19, C20, C21, C24, C25, C28, C29, C3, C30, C33, C34, C37, C38, C6, C7: value C -> 100nF
- C13, C14, C17, C18, C22, C23, C26, C27, C31, C32, C35, C36, C4, C5, C8, C9: value C -> 270nF
- Q1, Q10, Q11, Q12, Q13, Q14, Q15, Q16, Q2, Q3, Q4, Q5, Q6, Q7, Q8, Q9: footprint Package_TO_SOT_SMD:SOT-23-3 -> Package_TO_SOT_SMD:SOT-223
- R1, R11, R12, R2, R21, R22, R31, R32, R41, R42, R51, R52, R61, R62, R71, R72: value R_US -> 3Meg
- R10, R19, R20, R29, R30, R39, R40, R49, R50, R59, R60, R69, R70, R79, R80, R9: value R_US -> 5
- R13, R14, R23, R24, R3, R33, R34, R4, R43, R44, R53, R54, R63, R64, R73, R74: value R_US -> 470k
- R15, R16, R25, R26, R35, R36, R45, R46, R5, R55, R56, R6, R65, R66, R75, R76, R81, R82: value R_US -> 10k
- R17, R18, R27, R28, R37, R38, R47, R48, R57, R58, R67, R68, R7, R77, R78, R8: value R_US -> 1k
- moved H2 93.9 mm to (220.3, 68.2)
- moved H1 82.1 mm to (99.3, 68.0)
- moved H4 26.2 mm to (219.9, 125.8)
- moved R38 24.0 mm to (219.0, 83.8)
- moved R28 23.5 mm to (218.9, 91.3)
- moved R58 20.3 mm to (188.2, 83.8)
- moved R48 19.7 mm to (188.1, 91.3)
- moved R40 18.2 mm to (217.1, 79.7)
- moved R30 16.8 mm to (217.2, 87.2)
- moved R18 16.0 mm to (156.8, 83.8)
- moved R8 15.3 mm to (156.7, 91.3)
- moved Q8 15.0 mm to (211.8, 81.8), turned to 180 degrees
- moved J6 14.9 mm to (203.0, 69.8)
- moved J7 14.9 mm to (211.0, 74.8)
- moved J8 14.9 mm to (203.0, 74.8)
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Connections:
- J1 pad 26: unconnected-(J1-Pin_26-Pad26) -> +3.3V
- J1 pad 27: unconnected-(J1-Pin_27-Pad27) -> GND
- J10 pad 1: +3.3V -> Vdrive
- J11 pad 1: +3.3V -> Vdrive
- J12 pad 1: +3.3V -> Vdrive
- J13 pad 1: +3.3V -> Vdrive
- J14 pad 1: +3.3V -> Vdrive
- J15 pad 1: +3.3V -> Vdrive
- J16 pad 1: +3.3V -> Vdrive
- J17 pad 1: +3.3V -> Vdrive
- J18 pad 1: +3.3V -> Vdrive
- J2 pad 1: +3.3V -> Vdrive
- J3 pad 1: +3.3V -> Vdrive
- J4 pad 1: +3.3V -> Vdrive
- J5 pad 1: +3.3V -> Vdrive
- J6 pad 1: +3.3V -> Vdrive
- J7 pad 1: +3.3V -> Vdrive
- J8 pad 1: +3.3V -> Vdrive
- J9 pad 1: +3.3V -> Vdrive
- Q1 pad 1: Net-(J2-Pin_2) -> Net-(Q1-G)
- Q1 pad 2: Net-(Q1-G) -> Net-(J2-Pin_2)
- Q10 pad 1: Net-(J11-Pin_2) -> Net-(Q10-G)
- Q10 pad 2: Net-(Q10-G) -> Net-(J11-Pin_2)
- Q11 pad 1: Net-(J12-Pin_2) -> Net-(Q11-G)
- Q11 pad 2: Net-(Q11-G) -> Net-(J12-Pin_2)
- Q12 pad 1: Net-(J13-Pin_2) -> Net-(Q12-G)
- Q12 pad 2: Net-(Q12-G) -> Net-(J13-Pin_2)
- Q13 pad 1: Net-(J14-Pin_2) -> Net-(Q13-G)
- Q13 pad 2: Net-(Q13-G) -> Net-(J14-Pin_2)
- Q14 pad 1: Net-(J15-Pin_2) -> Net-(Q14-G)
- Q14 pad 2: Net-(Q14-G) -> Net-(J15-Pin_2)
- Q15 pad 1: Net-(J16-Pin_2) -> Net-(Q15-G)
- Q15 pad 2: Net-(Q15-G) -> Net-(J16-Pin_2)
- Q16 pad 1: Net-(J17-Pin_2) -> Net-(Q16-G)
- Q16 pad 2: Net-(Q16-G) -> Net-(J17-Pin_2)
- Q2 pad 1: Net-(J3-Pin_2) -> Net-(Q2-G)
- Q2 pad 2: Net-(Q2-G) -> Net-(J3-Pin_2)
- Q3 pad 1: Net-(J4-Pin_2) -> Net-(Q3-G)
- Q3 pad 2: Net-(Q3-G) -> Net-(J4-Pin_2)
- Q4 pad 1: Net-(J5-Pin_2) -> Net-(Q4-G)
- Q4 pad 2: Net-(Q4-G) -> Net-(J5-Pin_2)
- Q5 pad 1: Net-(J6-Pin_2) -> Net-(Q5-G)
- Q5 pad 2: Net-(Q5-G) -> Net-(J6-Pin_2)
- Q6 pad 1: Net-(J7-Pin_2) -> Net-(Q6-G)
- Q6 pad 2: Net-(Q6-G) -> Net-(J7-Pin_2)
- Q7 pad 1: Net-(J8-Pin_2) -> Net-(Q7-G)
- Q7 pad 2: Net-(Q7-G) -> Net-(J8-Pin_2)
- Q8 pad 1: Net-(J9-Pin_2) -> Net-(Q8-G)
- Q8 pad 2: Net-(Q8-G) -> Net-(J9-Pin_2)
- Q9 pad 1: Net-(J10-Pin_2) -> Net-(Q9-G)
- Q9 pad 2: Net-(Q9-G) -> Net-(J10-Pin_2)
Routing:
- net +3.3V: track 61.0 -> 164.5 mm, vias 8 -> 14
- net GND: track 83.5 -> 119.8 mm, vias 46 -> 52
- net Vdrive: track 0.00 -> 20.0 mm
- net /Quad_Current_Driver/I_SNS_3: track 18.8 -> 38.1 mm
- net /Quad_Current_Driver1/I_SNS_3: track 18.8 -> 37.9 mm
- net /Quad_Current_Driver3/I_SNS_3: track 18.8 -> 37.9 mm
- net /Quad_Current_Driver2/I_SNS_3: track 18.8 -> 37.8 mm
- net /bus1.PWM_SP3: track 119.4 -> 137.8 mm, vias 2 -> 4
- net /bus1.PWM_SP1: track 89.9 -> 107.3 mm
- net Net-(J4-Pin_2): track 8.25 -> 23.5 mm, vias 0 -> 2
- net Net-(J12-Pin_2): track 8.25 -> 23.5 mm, vias 0 -> 2
- net Net-(J16-Pin_2): track 8.25 -> 23.5 mm, vias 0 -> 2
- net Net-(J8-Pin_2): track 8.25 -> 23.5 mm, vias 0 -> 2
- net Net-(J3-Pin_2): track 8.74 -> 23.6 mm
- net Net-(J11-Pin_2): track 8.74 -> 23.6 mm
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- added copper zone on F.Cu, net Vdrive
- removed copper zone on F.Cu, net +3.3V
Other:
- board size 108.6 x 58.4 mm -> 129.4 x 66.2 mm
