File: SMA_Test_Bed/SMA_Test_Bed.kicad_sch (KiCad schematic)
At the start: 5 parts, among them J1 Conn_02x14_Counter_Clockwise, J18 Conn_01x02_Socket, U1 PCA9685PW

Commit message: Layout draft complete
Parts:
- added H1, H2, H3, H4: MountingHole, MountingHole:MountingHole_2.7mm_Pad_Via, symbol Mechanical:MountingHole
- added R81, R82: R_US, Resistor_SMD:R_0603_1608Metric, symbol Device:R_US
Connections:
- net +3.3V: now also R81.1, R82.2
- net SCL: now also R81.2
- net SDA: now also R82.1
Other:
- moved on the sheet: C1, C2, J1, J18, U1

Commit message: Added passive values
Parts:
- R81, R82: value R_US -> 10k
Changed lines of the file:
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@@
 			)
 		)
-		(property "Value" "R_US"
+		(property "Value" "10k"
 			(at 219.71 59.6899 0)
 			(effects
@@
 			)
 		)
-		(property "Value" "R_US"
+		(property "Value" "10k"
 			(at 231.14 59.6899 0)
 			(effects

Commit message: Time of fabrication
Parts:
- C1: Digikey PN (none) -> 490-14467-1-ND
- C2: Digikey PN (none) -> 311-1088-1-ND
- J1: Digikey PN (none) -> SSW-114-01-G-S-LL-ND
- R81, R82: Digikey PN (none) -> 311-10.0KHRCT-ND
- U1: Digikey PN (none) -> 568-5931-1-ND
Connections:
- net +3.3V: now also J1.26 (Pin_26); no longer J18.1 (Pin_1)
- net GND: now also J1.27 (Pin_27)
- new net Vdrive: J18.1 (Pin_1)
- no-connect marks 24 -> 22
